Commit message: adds velodyne, 2d pointcloud converter

File: spot_description/urdf/spot.urdf.xacro (robot description, xacro)
@@ -88,3 +88,7 @@
   <xacro:caster prefix="back_right" reflectH="-1" reflectV="-1"/>
   <xacro:include filename="$(find spot_description)/urdf/spot.plugins.xacro"/>
+  <xacro:include filename="$(find velodyne_description)/urdf/VLP-16.urdf.xacro"/>
+  <VLP-16 parent="base_footprint" name="velodyne" topic="lidar_points" hz="10" samples="1024" gpu="false" lasers="16" max_range="100">
+    <origin xyz="0 0 0.73" rpy="0 0 0" />
+  </VLP-16>
 </robot>

Commit message: Update master with spot simulation, navigation (#1)
* init commits for grpc base

* missing fields

* compiles the auth.proto from SDK!

* minimalist compilation example in c++

* Adds framework for Spot API Authentication using gRPC with a client and server

* adds velodyne, 2d pointcloud converter

* adds basic slam in the ahg apartment environment

* refactors a bit of the slam code. Adds navigation and AMCL localization abilities in addition to slam

* auth client and server run

* readded method

* adds ability to compile without grpc installed

Co-authored-by: Daksh <duadaksh@gmail.com>
Co-authored-by: Marika <marikamurphy@gmail.com>

File: spot_description/urdf/spot.urdf.xacro (robot description, xacro)
@@ -37,5 +37,5 @@
       <origin xyz="0 0 .655" rpy="0 0 0" />
       <geometry>
-        <mesh filename="$(find spot_description)/meshes/spot_whole_body.dae" />
+	      <mesh filename="package://spot_description/meshes/spot_whole_body.dae" />
       </geometry>
     </visual>
@@ -43,5 +43,5 @@
       <origin xyz="0 0 .655" rpy="0 0 0" />
       <geometry>
-        <mesh filename="$(find spot_description)/meshes/spot_whole_body.dae" />
+	      <mesh filename="package://spot_description/meshes/spot_whole_body.dae" />
       </geometry>
     </collision>
@@ -88,3 +88,7 @@
   <xacro:caster prefix="back_right" reflectH="-1" reflectV="-1"/>
   <xacro:include filename="$(find spot_description)/urdf/spot.plugins.xacro"/>
+  <xacro:include filename="$(find velodyne_description)/urdf/VLP-16.urdf.xacro"/>
+  <VLP-16 parent="base_footprint" name="velodyne" topic="lidar_points" hz="10" samples="1024" gpu="false" lasers="16" max_range="100">
+    <origin xyz="0 0 0.73" rpy="0 0 0" />
+  </VLP-16>
 </robot>
