Commit message: Cleaned up spot xacro code and made the physics more realistic (spot is no longer floating and invisible collisions have been minimized. Also fixed various roslaunch errors.

File: spot_description/urdf/spot.plugins.xacro (robot description, xacro)
@@ -3,5 +3,5 @@
   <!--Gazebo Differential Drive Plugin-->
   <gazebo>
-    <plugin name="differential_drive_controller" filename="libgazebo_ros_diff_drive.so">
+    <plugin name="diff_drive_controller" filename="libgazebo_ros_diff_drive.so">
       <alwaysOn>true</alwaysOn>
       <legacyMode>false</legacyMode>

File: spot_description/urdf/spot.urdf.xacro (robot description, xacro)
@@ -4,4 +4,5 @@
   <xacro:property name="wheel_separation" value="0.335"/>
   <xacro:property name="caster_wheel_radius" value="${wheel_radius/2}"/>
+  <xacro:property name="caster_wheel_mass" value="0.001"/>
   <xacro:property name="caster_wheel_joint_offset" value="0.3"/>
   <xacro:property name="wheel_offset" value="0.025"/>
@@ -54,5 +55,5 @@
         </geometry>
       </collision>
-      <xacro:cylinder_inertia m="0.05" r="${wheel_radius}" h="0.005"/>
+      <xacro:cylinder_inertia m="0.5" r="${wheel_radius}" h="0.005"/>
     </link>
     <joint name="${prefix}_wheel_joint" type="continuous">
@@ -63,6 +64,6 @@
     </joint>
   </xacro:macro>
-  <xacro:wheel prefix="left" reflect="0.8"/>
-  <xacro:wheel prefix="right" reflect="-0.8"/>
+  <xacro:wheel prefix="left" reflect="0.6"/>
+  <xacro:wheel prefix="right" reflect="-0.6"/>
   <xacro:macro name="caster" params="prefix reflectH reflectV">
     <link name="${prefix}_caster_wheel">
@@ -73,5 +74,5 @@
         </geometry>
       </collision>
-      <xacro:sphere_inertia m="0.001" r="${caster_wheel_radius}"/>
+      <xacro:sphere_inertia m="0.05" r="${caster_wheel_radius}"/>
     </link>
     <joint name="${prefix}_caster_wheel_joint" type="continuous">

Commit message: adds basic slam in the ahg apartment environment

File: spot_description/urdf/spot.plugins.xacro (robot description, xacro)
@@ -4,4 +4,6 @@
   <gazebo>
     <plugin name="diff_drive_controller" filename="libgazebo_ros_diff_drive.so">
+      <publishWheelTF>true</publishWheelTF>
+      <publishOdomTF>true</publishOdomTF>
       <alwaysOn>true</alwaysOn>
       <legacyMode>false</legacyMode>

File: spot_description/urdf/spot.urdf.xacro (robot description, xacro)
@@ -37,5 +37,5 @@
       <origin xyz="0 0 .655" rpy="0 0 0" />
       <geometry>
-        <mesh filename="$(find spot_description)/meshes/spot_whole_body.dae" />
+	      <mesh filename="package://spot_description/meshes/spot_whole_body.dae" />
       </geometry>
     </visual>
@@ -43,5 +43,5 @@
       <origin xyz="0 0 .655" rpy="0 0 0" />
       <geometry>
-        <mesh filename="$(find spot_description)/meshes/spot_whole_body.dae" />
+	      <mesh filename="package://spot_description/meshes/spot_whole_body.dae" />
       </geometry>
     </collision>

Commit message: camera model added

File: spot_description/urdf/spot.plugins.xacro (robot description, xacro)
@@ -20,3 +20,46 @@
     </plugin>
   </gazebo>
+   <gazebo reference="camera_rgb_frame">
+    <sensor type="depth" name="realsense_R200">
+      <always_on>true</always_on>
+      <visualize>false</visualize>
+      <camera>
+          <horizontal_fov>1.3439</horizontal_fov>
+          <image>
+              <width>1920</width>
+              <height>1080</height>
+              <format>R8G8B8</format>
+          </image>
+          <depth_camera></depth_camera>
+          <clip>
+              <near>0.03</near>
+              <far>100</far>
+          </clip>
+      </camera>
+      <plugin name="camera_controller" filename="libgazebo_ros_openni_kinect.so">
+        <baseline>0.2</baseline>
+        <alwaysOn>true</alwaysOn>
+        <updateRate>30.0</updateRate>
+        <cameraName>camera</cameraName>
+        <frameName>camera_link</frameName>
+        <imageTopicName>rgb/image_raw</imageTopicName>
+        <depthImageTopicName>depth/image_raw</depthImageTopicName>
+        <pointCloudTopicName>depth/points</pointCloudTopicName>
+        <cameraInfoTopicName>rgb/camera_info</cameraInfoTopicName>
+        <depthImageCameraInfoTopicName>depth/camera_info</depthImageCameraInfoTopicName>
+        <pointCloudCutoff>0.4</pointCloudCutoff>
+            <hackBaseline>0.07</hackBaseline>
+            <distortionK1>0.0</distortionK1>
+            <distortionK2>0.0</distortionK2>
+            <distortionK3>0.0</distortionK3>
+            <distortionT1>0.0</distortionT1>
+            <distortionT2>0.0</distortionT2>
+        <CxPrime>0.0</CxPrime>
+        <Cx>0.0</Cx>
+        <Cy>0.0</Cy>
+        <focalLength>0</focalLength>
+        <hackBaseline>0</hackBaseline>
+      </plugin>
+    </sensor>
+  </gazebo>
 </robot>

File: spot_description/urdf/spot.urdf.xacro (robot description, xacro)
@@ -87,8 +87,33 @@
   <xacro:caster prefix="back_left" reflectH="1" reflectV="-1"/>
   <xacro:caster prefix="back_right" reflectH="-1" reflectV="-1"/>
-  <xacro:include filename="$(find spot_description)/urdf/spot.plugins.xacro"/>
+  <joint name="camera_joint" type="fixed">
+    <origin xyz="0.425 -0.065 0.63" rpy="0 0 0"/>
+    <parent link="base_footprint"/>
+    <child link="camera_link"/>
+  </joint>
+  <link name="camera_link">
+    <visual>
+     <origin xyz="0 0 0" rpy="1.57 0 1.57"/>
+      <geometry>
+       <mesh filename="package://spot_description/meshes/r200.dae" />
+      </geometry>
+    </visual>
+    <collision>
+      <origin xyz="0.003 0.065 0.007" rpy="0 0 0"/>
+      <geometry>
+        <box size="0.012 0.132 0.020"/>
+      </geometry>
+    </collision>
+  </link>
+  <joint name="camera_rgb_joint" type="fixed">
+    <origin xyz="0.005 0.018 0.013" rpy="0 0 0"/>
+    <parent link="camera_link"/>
+    <child link="camera_rgb_frame"/>
+  </joint>
+  <link name="camera_rgb_frame"/>
   <xacro:include filename="$(find velodyne_description)/urdf/VLP-16.urdf.xacro"/>
   <VLP-16 parent="base_footprint" name="velodyne" topic="lidar_points" hz="10" samples="1024" gpu="false" lasers="16" max_range="100">
     <origin xyz="0 0 0.73" rpy="0 0 0" />
   </VLP-16>
+  <xacro:include filename="$(find spot_description)/urdf/spot.plugins.xacro"/>
 </robot>

File: spot_description/urdf/spot.xacro (robot description, xacro)
@@ -82,4 +82,29 @@
     </joint>
   </xacro:macro>
+  <joint name="camera_joint" type="fixed">
+    <origin xyz="0.064 -0.065 0.154" rpy="0 0 0"/>
+    <parent link="base_footprint"/>
+    <child link="camera_link"/>
+  </joint>
+  <link name="camera_link">
+    <visual>
+     <origin xyz="0 0 0" rpy="1.57 0 1.57"/>
+      <geometry>
+       <mesh filename="$(find spot_description)/meshes/r200.dae" />
+      </geometry>
+    </visual>
+    <collision>
+      <origin xyz="0.003 0.065 0.007" rpy="0 0 0"/>
+      <geometry>
+        <box size="0.012 0.132 0.020"/>
+      </geometry>
+    </collision>
+  </link>
+  <joint name="camera_rgb_joint" type="fixed">
+    <origin xyz="$0.005 0.018 0.013" rpy="0 0 0"/>
+    <parent link="camera_link"/>
+    <child link="camera_rgb_frame"/>
+  </joint>
+  <link name="camera_rgb_frame"/>
   <xacro:caster prefix="front_left" reflectH="1" reflectV="1"/>
   <xacro:caster prefix="front_right" reflectH="-1" reflectV="1"/>
