Commit message: renamed spot_description package

File: spot_description/urdf/spot.urdf (robot description, URDF)
Before this commit: robot spot, 13 links, 12 joints
Links:
- link base: geometry collision mesh filename=package://spot_sim_description/meshes/base.dae; visual mesh filename=package://spot_sim_description/meshes/base.dae
- link fl.hip: geometry collision mesh filename=package://spot_sim_description/meshes/fl.hip.dae; visual mesh filename=package://spot_sim_description/meshes/fl.hip.dae
- link fl.lleg: geometry collision mesh filename=package://spot_sim_description/meshes/fl.lleg.dae; visual mesh filename=package://spot_sim_description/meshes/fl.lleg.dae
- link fl.uleg: geometry collision mesh filename=package://spot_sim_description/meshes/fl.uleg.dae; visual mesh filename=package://spot_sim_description/meshes/fl.uleg.dae
- link fr.hip: geometry collision mesh filename=package://spot_sim_description/meshes/fr.hip.dae; visual mesh filename=package://spot_sim_description/meshes/fr.hip.dae
- link fr.lleg: geometry collision mesh filename=package://spot_sim_description/meshes/fr.lleg.dae; visual mesh filename=package://spot_sim_description/meshes/fr.lleg.dae
- link fr.uleg: geometry collision mesh filename=package://spot_sim_description/meshes/fr.uleg.dae; visual mesh filename=package://spot_sim_description/meshes/fr.uleg.dae
- link hl.hip: geometry collision mesh filename=package://spot_sim_description/meshes/hl.hip.dae; visual mesh filename=package://spot_sim_description/meshes/hl.hip.dae
- link hl.lleg: geometry collision mesh filename=package://spot_sim_description/meshes/hl.lleg.dae; visual mesh filename=package://spot_sim_description/meshes/hl.lleg.dae
- link hl.uleg: geometry collision mesh filename=package://spot_sim_description/meshes/hl.uleg.dae; visual mesh filename=package://spot_sim_description/meshes/hl.uleg.dae
- link hr.hip: geometry collision mesh filename=package://spot_sim_description/meshes/hr.hip.dae; visual mesh filename=package://spot_sim_description/meshes/hr.hip.dae
- link hr.lleg: geometry collision mesh filename=package://spot_sim_description/meshes/hr.lleg.dae; visual mesh filename=package://spot_sim_description/meshes/hr.lleg.dae
- link hr.uleg: geometry collision mesh filename=package://spot_sim_description/meshes/hr.uleg.dae; visual mesh filename=package://spot_sim_description/meshes/hr.uleg.dae

File: spot_description/urdf/spot.urdf.xacro (robot description, xacro)
@@ -37,5 +37,5 @@
       <origin xyz="0 0 .655" rpy="0 0 0" />
       <geometry>
-	      <mesh filename="package://spot_description/meshes/spot_whole_body.dae" />
+	      <mesh filename="package://spot_sim_description/meshes/spot_whole_body.dae" />
       </geometry>
     </visual>
@@ -43,5 +43,5 @@
       <origin xyz="0 0 .655" rpy="0 0 0" />
       <geometry>
-	      <mesh filename="package://spot_description/meshes/spot_whole_body.dae" />
+	      <mesh filename="package://spot_sim_description/meshes/spot_whole_body.dae" />
       </geometry>
     </collision>
@@ -87,5 +87,5 @@
   <xacro:caster prefix="back_left" reflectH="1" reflectV="-1"/>
   <xacro:caster prefix="back_right" reflectH="-1" reflectV="-1"/>
-  <xacro:include filename="$(find spot_description)/urdf/spot.plugins.xacro"/>
+  <xacro:include filename="$(find spot_sim_description)/urdf/spot.plugins.xacro"/>
   <!--<xacro:include filename="$(find velodyne_description)/urdf/VLP-16.urdf.xacro"/>
   <VLP-16 parent="base_footprint" name="velodyne" topic="lidar_points" hz="10" samples="1024" gpu="false" lasers="16" max_range="100">

File: spot_description/urdf/spot.xacro (robot description, xacro)
@@ -36,5 +36,5 @@
       <origin xyz="0 0 .655" rpy="0 0 0" />
       <geometry>
-        <mesh filename="$(find spot_description)/meshes/spot_whole_body.dae" />
+        <mesh filename="$(find spot_sim_description)/meshes/spot_whole_body.dae" />
       </geometry>
     </visual>
@@ -42,5 +42,5 @@
       <origin xyz="0 0 .655" rpy="0 0 0" />
       <geometry>
-        <mesh filename="$(find spot_description)/meshes/spot_whole_body.dae" />
+        <mesh filename="$(find spot_sim_description)/meshes/spot_whole_body.dae" />
       </geometry>
     </collision>
@@ -86,4 +86,4 @@
   <xacro:caster prefix="back_left" reflectH="1" reflectV="-1"/>
   <xacro:caster prefix="back_right" reflectH="-1" reflectV="-1"/>
-  <xacro:include filename="$(find spot_description)/urdf/spot.plugins.xacro"/>
+  <xacro:include filename="$(find spot_sim_description)/urdf/spot.plugins.xacro"/>
 </robot>
