Commit message: rolled back velodyne package deletion

File: spot_sim_description/urdf/spot.urdf.xacro (robot description, xacro)
@@ -32,4 +32,5 @@
     </inertial>
   </xacro:macro>
+  <!-- <link name="base_footprint" /> -->
   <link name="base_footprint">
     <xacro:default_inertial mass="32.5"/>
@@ -89,6 +90,6 @@
   <xacro:include filename="$(find spot_sim_description)/urdf/spot.plugins.xacro"/>
   <xacro:include filename="$(find velodyne_description)/urdf/VLP-16.urdf.xacro"/>
-  <VLP-16 parent="base_footprint" name="velodyne" topic="lidar_points" hz="10" samples="1024" gpu="false" lasers="16" max_range="100">
+  <xacro:VLP-16 parent="base_footprint" name="velodyne" topic="/lidar_points" hz="10" samples="1024" gpu="false" lasers="16" max_range="100">
     <origin xyz="0 0 0.73" rpy="0 0 0" />
-  </VLP-16>
+  </xacro:VLP-16>
 </robot>
