Commit message: velodyne working in Gazebo, dependencies moved to package.xml for rosdep installation

File: spot_sim_description/urdf/spot.urdf (robot description, URDF)
Before this commit: robot spot, 13 links, 12 joints
Links:
- removed link base
- removed link fl.hip
- removed link fl.lleg
- removed link fl.uleg
- removed link fr.hip
- removed link fr.lleg
- removed link fr.uleg
- removed link hl.hip
- removed link hl.lleg
- removed link hl.uleg
- removed link hr.hip
- removed link hr.lleg
- removed link hr.uleg
- added link back_left_caster_wheel, mass 0.05; collision sphere radius=0.015
- added link back_right_caster_wheel, mass 0.05; collision sphere radius=0.015
- added link base_footprint
- added link base_link, mass 32.5; collision mesh filename=package://spot_sim_description/meshes/spot_whole_body.dae; visual mesh filename=package://spot_sim_description/meshes/spot_whole_body.dae
- added link left_wheel, mass 0.5; collision cylinder length=0.005 radius=0.03
- added link right_wheel, mass 0.5; collision cylinder length=0.005 radius=0.03
- added link velodyne, mass 0.01; visual mesh filename=package://velodyne_description/meshes/VLP16_scan.dae
- added link velodyne_base_link, mass 0.83; collision cylinder length=0.0717 radius=0.0516; visual mesh filename=package://velodyne_description/meshes/VLP16_base_1.dae
Joints:
- removed joint fl.hx
- removed joint fl.hy
- removed joint fl.kn
- removed joint fr.hx
- removed joint fr.hy
- removed joint fr.kn
- removed joint hl.hx
- removed joint hl.hy
- removed joint hl.kn
- removed joint hr.hx
- removed joint hr.hy
- removed joint hr.kn
- added joint back_left_caster_wheel_joint: type continuous, parent base_link, child back_left_caster_wheel, origin xyz=-0.27499999999999997 0.1675 -0.02 rpy=0 0 0, axis 0 1 0
- added joint back_right_caster_wheel_joint: type continuous, parent base_link, child back_right_caster_wheel, origin xyz=-0.27499999999999997 -0.1675 -0.02 rpy=0 0 0, axis 0 1 0
- added joint footprint: type fixed, parent base_footprint, child base_link, origin xyz=0 0 0.655 rpy=0 0 0
- added joint left_wheel_joint: type continuous, parent base_link, child left_wheel, origin xyz=0.025 0.1005 -0.005 rpy=0 0 0, axis 0 1 0
- added joint right_wheel_joint: type continuous, parent base_link, child right_wheel, origin xyz=0.025 -0.1005 -0.005 rpy=0 0 0, axis 0 1 0
- added joint velodyne_base_mount_joint: type fixed, parent base_link, child velodyne_base_link, origin xyz=0 0 0.73 rpy=0 0 0
- added joint velodyne_base_scan_joint: type fixed, parent velodyne_base_link, child velodyne, origin xyz=0 0 0.0377 rpy=0 0 0

File: spot_sim_description/urdf/spot.urdf.xacro (robot description, xacro)
@@ -32,17 +32,22 @@
     </inertial>
   </xacro:macro>
-  <!-- <link name="base_footprint" /> -->
-  <link name="base_footprint">
+  <link name="base_footprint" />
+  <joint name="footprint" type="fixed" >
+    <parent link="base_footprint" />
+    <child link="base_link" />
+    <origin xyz="0 0 0.655" rpy="0 0 0" />
+  </joint>
+  <link name="base_link">
     <xacro:default_inertial mass="32.5"/>
     <visual name="visual">
-      <origin xyz="0 0 .655" rpy="0 0 0" />
+      <origin xyz="0 0 0" rpy="0 0 0" />
       <geometry>
-	      <mesh filename="package://spot_sim_description/meshes/spot_whole_body.dae" />
+        <mesh filename="package://spot_sim_description/meshes/spot_whole_body.dae" />
       </geometry>
     </visual>
     <collision>
-      <origin xyz="0 0 .655" rpy="0 0 0" />
+      <origin xyz="0 0 0" rpy="0 0 0" />
       <geometry>
-	      <mesh filename="package://spot_sim_description/meshes/spot_whole_body.dae" />
+        <mesh filename="package://spot_sim_description/meshes/spot_whole_body.dae" />
       </geometry>
     </collision>
@@ -60,5 +65,5 @@
     <joint name="${prefix}_wheel_joint" type="continuous">
       <axis xyz="0 1 0" rpy="0 0 0" />
-      <parent link="base_footprint"/>
+      <parent link="base_link"/>
       <child link="${prefix}_wheel"/>
       <origin xyz="${wheel_offset} ${(wheel_separation/2)*reflect} -0.005" rpy="0 0 0"/>
@@ -79,5 +84,5 @@
     <joint name="${prefix}_caster_wheel_joint" type="continuous">
       <axis xyz="0 1 0" rpy="0 0 0" />
-      <parent link="base_footprint"/>
+      <parent link="base_link"/>
       <child link="${prefix}_caster_wheel"/>
       <origin xyz="${wheel_offset + caster_wheel_joint_offset*reflectV} ${wheel_separation/2*reflectH} -${caster_wheel_radius+0.005}" rpy="0 0 0"/>
@@ -90,5 +95,5 @@
   <xacro:include filename="$(find spot_sim_description)/urdf/spot.plugins.xacro"/>
   <xacro:include filename="$(find velodyne_description)/urdf/VLP-16.urdf.xacro"/>
-  <xacro:VLP-16 parent="base_footprint" name="velodyne" topic="/lidar_points" hz="10" samples="1024" gpu="false" lasers="16" max_range="100">
+  <xacro:VLP-16 parent="base_link" name="velodyne" topic="/lidar_points" hz="10" samples="1024" gpu="false" lasers="16" max_range="100">
     <origin xyz="0 0 0.73" rpy="0 0 0" />
   </xacro:VLP-16>
